File: beacon.kicad/beacon.kicad_pcb (KiCad board)
At the start: 2 copper layers, 0 parts

Commit message: libs for RP2354A, ABM8-272-T3 and AOTA-B201610S3R3-101-T
Parts:
- added L1: AOTA-B201610S3R3-101-T, AOTA-B201610S3R3-101-T:AOTAB201610S3R3101T, F.Cu at (63.5, 61.3)
- added U1: RP2354A, RP2354A:RP2354A-QFN-60-1EP_7x7mm_P0.4mm_EP3.4x3.4mm, F.Cu at (53.5, 58.4)
- added Y1: ABM8-272-T3, ABM8-272-T3:ABM8272T3, F.Cu at (63.8, 56.0)

Commit message: schematic draft
Parts:
- added C1: 10u, Capacitor_SMD:C_0805_2012Metric, F.Cu at (79.9, 65.5)
- added C10: 4.7u, Capacitor_SMD:C_0805_2012Metric, F.Cu at (72.4, 84.0)
- added C11: 100n, Capacitor_SMD:C_0805_2012Metric, F.Cu at (72.4, 87.0)
- added C12: 100n, Capacitor_SMD:C_0805_2012Metric, F.Cu at (72.4, 90.0)
- added C13: 100n, Capacitor_SMD:C_0805_2012Metric, F.Cu at (72.4, 93.0)
- added C14: 100n, Capacitor_SMD:C_0805_2012Metric, F.Cu at (72.4, 96.0)
- added C15: 100n, Capacitor_SMD:C_0805_2012Metric, F.Cu at (76.8, 81.0)
- added C16: 100n, Capacitor_SMD:C_0805_2012Metric, F.Cu at (76.8, 84.0)
- added C17: 100n, Capacitor_SMD:C_0805_2012Metric, F.Cu at (76.8, 87.0)
- added C18: 100n, Capacitor_SMD:C_0805_2012Metric, F.Cu at (76.8, 90.0)
- added C19: 10u, Capacitor_SMD:C_0805_2012Metric, F.Cu at (76.8, 93.0)
- added C3: 15p, Capacitor_SMD:C_0805_2012Metric, F.Cu at (69.4, 47.8)
- added C4: 15p, Capacitor_SMD:C_0805_2012Metric, F.Cu at (69.4, 51.2)
- added C5: 10u, Capacitor_SMD:C_0805_2012Metric, F.Cu at (79.9, 68.5)
- added C6: 4.7u, Capacitor_SMD:C_0805_2012Metric, F.Cu at (85.8, 55.8)
- added C7: 4.7u, Capacitor_SMD:C_0805_2012Metric, F.Cu at (85.8, 58.8)
- added C8: 100n, Capacitor_SMD:C_0805_2012Metric, F.Cu at (72.4, 81.0)
- added C9: 4.7u, Capacitor_SMD:C_0805_2012Metric, F.Cu at (85.8, 61.8)
- added D1: SK6812, LED_SMD:LED_SK6812_PLCC4_5.0x5.0mm_P3.2mm, F.Cu at (83.1, 82.8)
- added J1: USB, Connector_PinHeader_1.27mm:PinHeader_1x05_P1.27mm_Horizontal, F.Cu at (73.2, 54.5)
- added J2: SWD, Connector_PinHeader_1.27mm:PinHeader_1x03_P1.27mm_Horizontal, F.Cu at (70.8, 68.4)
- added R1: 5k1, Resistor_SMD:R_0805_2012Metric, F.Cu at (79.9, 71.5)
- added R2: 1k, Resistor_SMD:R_0805_2012Metric, F.Cu at (69.4, 54.5)
- added R5: 33, Resistor_SMD:R_0805_2012Metric, F.Cu at (90.2, 61.6)
- added R7: 27, Resistor_SMD:R_0805_2012Metric, F.Cu at (90.2, 58.7)
- added R8: 27, Resistor_SMD:R_0805_2012Metric, F.Cu at (90.2, 55.7)
- added U2: NCP1117-3.3_SOT223, Package_TO_SOT_SMD:SOT-223-3_TabPin2, F.Cu at (58.6, 70.3)
Connections:
- L1 pad 1: unconnected-(L1-Pad1) -> +1V1
- L1 pad 2: unconnected-(L1-Pad2) -> /VREG_LX
- U1 pad 1: Net-(U1-IOVDD-Pad1) -> +3V3
- U1 pad 11: Net-(U1-IOVDD-Pad1) -> +3V3
- U1 pad 20: Net-(U1-IOVDD-Pad1) -> +3V3
- U1 pad 21: unconnected-(U1-XIN-Pad21) -> /XIN
- U1 pad 22: unconnected-(U1-XOUT-Pad22) -> /XOUT
- U1 pad 23: Net-(U1-DVDD-Pad23) -> +1V1
- U1 pad 24: unconnected-(U1-SWCLK-Pad24) -> /SWCLK
- U1 pad 25: unconnected-(U1-SWDIO-Pad25) -> /SWDIO
- U1 pad 30: Net-(U1-IOVDD-Pad1) -> +3V3
- U1 pad 38: Net-(U1-IOVDD-Pad1) -> +3V3
- U1 pad 39: Net-(U1-DVDD-Pad23) -> +1V1
- U1 pad 42: unconnected-(U1-GPIO28/ADC2-Pad42) -> /RGB_DIN
- U1 pad 44: unconnected-(U1-ADC_AVDD-Pad44) -> +3V3
- U1 pad 45: Net-(U1-IOVDD-Pad1) -> +3V3
- U1 pad 46: unconnected-(U1-VREG_AVDD-Pad46) -> /VREG_AVDD
- U1 pad 47: unconnected-(U1-VREG_PGND-Pad47) -> GND
- U1 pad 48: unconnected-(U1-VREG_LX-Pad48) -> /VREG_LX
- U1 pad 49: unconnected-(U1-VREG_VIN-Pad49) -> +3V3
- U1 pad 50: unconnected-(U1-VREG_FB-Pad50) -> +1V1
- U1 pad 51: unconnected-(U1-USB_DM-Pad51) -> Net-(U1-USB_DM)
- U1 pad 52: unconnected-(U1-USB_DP-Pad52) -> Net-(U1-USB_DP)
- U1 pad 53: unconnected-(U1-USB_OTP_VDD-Pad53) -> +3V3
- U1 pad 54: unconnected-(U1-QSPI_IOVDD-Pad54) -> +3V3
- U1 pad 6: Net-(U1-DVDD-Pad23) -> +1V1
- U1 pad 61: unconnected-(U1-GND-Pad61) -> GND
- Y1 pad 1: unconnected-(Y1-CRYSTAL_1-Pad1) -> /XIN
- Y1 pad 2: unconnected-(Y1-GND_1-Pad2) -> GND
- Y1 pad 3: unconnected-(Y1-CRYSTAL_2-Pad3) -> Net-(Y1-CRYSTAL_2)
- Y1 pad 4: unconnected-(Y1-GND_2-Pad4) -> GND

Commit message: initial PoC design
Parts:
- added R3: 500, Resistor_SMD:R_0805_2012Metric, F.Cu at (139.5, 95.8)
- C6, C7: footprint Capacitor_SMD:C_0805_2012Metric -> RP2354A:C_0402_1005Metric_small_pads
- C9: footprint Capacitor_SMD:C_0805_2012Metric -> Capacitor_SMD:C_0402_1005Metric
- R1, R5, R7, R8: footprint Resistor_SMD:R_0805_2012Metric -> Resistor_SMD:R_0402_1005Metric
- U1: footprint RP2354A:RP2354A-QFN-60-1EP_7x7mm_P0.4mm_EP3.4x3.4mm -> RP2354A:RP2354A-QFN-60-1EP_7x7_P0.4mm_EP3.4x3.4mm_ThermalVias
- moved U1 101.7 mm to (144.3, 104.3)
- moved C4 97.9 mm to (147.3, 110.4), turned to 90 degrees
- moved Y1 96.5 mm to (141.9, 112.7)
- moved C3 94.9 mm to (138.7, 112.6), turned to -90 degrees
- moved U2 92.2 mm to (148.3, 91.6), turned to -90 degrees
- moved R2 91.8 mm to (142.6, 109.8)
- moved J2 90.9 mm to (149.9, 113.1), turned to -90 degrees
- moved L1 90.2 mm to (146.3, 97.1)
- moved C11 79.6 mm to (150.3, 103.2)
- moved C14 78.4 mm to (150.3, 105.1)
- moved C10 77.6 mm to (145.3, 110.4), turned to -90 degrees
- moved C5 77.2 mm to (151.0, 98.5), turned to -90 degrees
- moved C16 77.0 mm to (150.3, 107.1)
- moved C19 75.2 mm to (150.3, 109.0)
- moved C17 74.8 mm to (150.3, 101.2)
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Connections:
- D1 pad 2: /RGB_DIN -> Net-(D1-DIN)
- J1 pad 1: VBUS -> GND
- J1 pad 2: /USB_D- -> /USB_CC
- J1 pad 4: /USB_CC -> /USB_D-
- J1 pad 5: GND -> VBUS
- J2 pad 1: /SWCLK -> /SWDIO
- J2 pad 3: /SWDIO -> /SWCLK
- U1 pad 2: unconnected-(U1-GPIO0-Pad2) -> /RGB_DIN
- U1 pad 42: /RGB_DIN -> unconnected-(U1-GPIO28/ADC2-Pad42)
Routing:
- net +3V3: track 0.00 -> 31.1 mm, vias 0 -> 2
- net GND: track 0.00 -> 30.6 mm, vias 0 -> 16
- net +1V1: track 0.00 -> 19.1 mm, vias 0 -> 9
- net /USB_D-: track 0.00 -> 12.4 mm
- net /USB_D+: track 0.00 -> 12.4 mm
- net /XIN: track 0.00 -> 10.4 mm
- net /SWDIO: track 0.00 -> 9.16 mm
- net /SWCLK: track 0.00 -> 9.06 mm
- net /RGB_DIN: track 0.00 -> 8.50 mm
- net Net-(Y1-CRYSTAL_2): track 0.00 -> 7.24 mm
- net /USB_CC: track 0.00 -> 4.23 mm
- net /VREG_AVDD: track 0.00 -> 3.56 mm
- net Net-(U1-USB_DM): track 0.00 -> 2.83 mm
- net Net-(D1-DIN): track 0.00 -> 2.68 mm
- net Net-(U1-USB_DP): track 0.00 -> 2.58 mm
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- added copper zone on F.Cu, net +1V1
- added copper zone on F.Cu, net +3V3
- added copper zone on F.Cu, net /VREG_LX
- added copper zone on B.Cu, net GND
- added copper zone on F.Cu, net GND
- added copper zone on F.Cu, net VBUS
Other:
- board outline added: 14.8 x 30.4 mm
