File: beacon.kicad/beacon.kicad_sch (KiCad schematic)
At the start: 0 parts

Commit message: libs for RP2354A, ABM8-272-T3 and AOTA-B201610S3R3-101-T
Parts:
- added L1: AOTA-B201610S3R3-101-T, AOTA-B201610S3R3-101-T:AOTAB201610S3R3101T, symbol AOTA-B201610S3R3-101-T:AOTA-B201610S3R3-101-T
- added U1: RP2354A, RP2354A:RP2354A-QFN-60-1EP_7x7mm_P0.4mm_EP3.4x3.4mm, symbol MCU_RaspberryPi:RP2354A
- added Y1: ABM8-272-T3, ABM8-272-T3:ABM8272T3, symbol ABM8-272-T3:ABM8-272-T3
Connections:
- new net: U1.1 (IOVDD), U1.11 (IOVDD), U1.20 (IOVDD), U1.30 (IOVDD), U1.38 (IOVDD), U1.45 (IOVDD)
- new net: U1.23 (DVDD), U1.39 (DVDD), U1.6 (DVDD)

Commit message: schematic draft
Parts:
- added C1, C5: 10u, Capacitor_SMD:C_0805_2012Metric, symbol Device:C
- added C10, C6, C7, C9: 4.7u, Capacitor_SMD:C_0805_2012Metric, symbol Device:C_Small
- added C11, C12, C13, C14, C15, C16, C17, C18, C8: 100n, Capacitor_SMD:C_0805_2012Metric, symbol Device:C_Small
- added C19: 10u, Capacitor_SMD:C_0805_2012Metric, symbol Device:C_Small
- added C3, C4: 15p, Capacitor_SMD:C_0805_2012Metric, symbol Device:C_Small
- added D1: SK6812, LED_SMD:LED_SK6812_PLCC4_5.0x5.0mm_P3.2mm, symbol LED:SK6812
- added J1: USB, Connector_PinHeader_1.27mm:PinHeader_1x05_P1.27mm_Horizontal, symbol Connector_Generic:Conn_01x05
- added J2: SWD, Connector_PinHeader_1.27mm:PinHeader_1x03_P1.27mm_Horizontal, symbol Connector_Generic:Conn_01x03
- added R1: 5k1, Resistor_SMD:R_0805_2012Metric, symbol Device:R_Small
- added R2: 1k, Resistor_SMD:R_0805_2012Metric, symbol Device:R_Small
- added R5: 33, Resistor_SMD:R_0805_2012Metric, symbol Device:R_Small
- added R7, R8: 27, Resistor_SMD:R_0805_2012Metric, symbol Device:R_Small
- added U2: NCP1117-3.3_SOT223, Package_TO_SOT_SMD:SOT-223-3_TabPin2, symbol Regulator_Linear:NCP1117-3.3_SOT223
Connections:
- net XIN: now reaches Y1.1 (CRYSTAL_1)
- net XIN: now also U1.21 (XIN), C3.1
- net GND: now reaches Y1.2 (GND_1)
- net GND: now also U1.47 (VREG_PGND), U1.61 (GND), Y1.4 (GND_2), C1.2, C10.2, C11.2, C12.2, C13.2, C14.2, C15.2, C16.2, C17.2, C18.2, C19.2, C3.2, C4.2, C5.2, C6.2, C7.2, C8.2, C9.2, D1.1 (VSS), J1.5 (Pin_5), J2.2 (Pin_2), R1.1, U2.1 (GND)
- net at Y1.3 (CRYSTAL_2): now also C4.1, R2.1
- net +1V1: now reaches L1.1
- net +1V1: now also U1.23 (DVDD), U1.39 (DVDD), U1.50 (VREG_FB), U1.6 (DVDD), C10.1, C11.1, C7.1, C8.1
- net VREG_LX: now reaches L1.2
- net VREG_LX: now also U1.48 (VREG_LX)
- net +3V3: now reaches U1.1 (IOVDD), U1.11 (IOVDD), U1.20 (IOVDD), U1.30 (IOVDD), U1.38 (IOVDD), U1.45 (IOVDD)
- net +3V3: now also U1.44 (ADC_AVDD), U1.49 (VREG_VIN), U1.53 (USB_OTP_VDD), U1.54 (QSPI_IOVDD), C12.1, C13.1, C14.1, C15.1, C16.1, C17.1, C18.1, C19.1, C5.1, C6.1, D1.3 (VDD), R5.1, U2.2 (VO)
- net XOUT: now reaches U1.22 (XOUT)
- net XOUT: now also R2.2
- net SWCLK: now reaches U1.24 (SWCLK)
- net SWCLK: now also J2.1 (Pin_1)
- net SWDIO: now reaches U1.25 (SWDIO)
- net SWDIO: now also J2.3 (Pin_3)
- net RGB_DIN: now reaches U1.42 (GPIO28/ADC2)
- net RGB_DIN: now also D1.2 (DIN)
- net VREG_AVDD: now reaches U1.46 (VREG_AVDD)
- net VREG_AVDD: now also C9.1, R5.2
- net at U1.51 (USB_DM): now also R8.2
- net at U1.52 (USB_DP): now also R7.2
- new net USB_CC: J1.4 (Pin_4), R1.2
- new net USB_D+: J1.3 (Pin_3), R7.1
- new net USB_D-: J1.2 (Pin_2), R8.1
- new net VBUS: C1.1, J1.1 (Pin_1), U2.3 (VI)
- no-connect marks 0 -> 37
Other:
- note added: "12MHz"
- note added: "Debug"
- note added: "USB / Power"
- note added: "VREG"
- moved on the sheet: L1, U1, Y1

Commit message: initial PoC design
Parts:
- added R3: 500, Resistor_SMD:R_0805_2012Metric, symbol Device:R_Small
- C6, C7: footprint Capacitor_SMD:C_0805_2012Metric -> RP2354A:C_0402_1005Metric_small_pads
- C9: footprint Capacitor_SMD:C_0805_2012Metric -> Capacitor_SMD:C_0402_1005Metric
- R1, R5, R7, R8: footprint Resistor_SMD:R_0805_2012Metric -> Resistor_SMD:R_0402_1005Metric
- U1: footprint RP2354A:RP2354A-QFN-60-1EP_7x7mm_P0.4mm_EP3.4x3.4mm -> RP2354A:RP2354A-QFN-60-1EP_7x7_P0.4mm_EP3.4x3.4mm_ThermalVias
Connections:
- net GND: now also J1.1 (Pin_1); no longer J1.5 (Pin_5)
- net RGB_DIN: now also U1.2 (GPIO0), R3.1; no longer D1.2 (DIN), U1.42 (GPIO28/ADC2)
- net SWCLK: now also J2.3 (Pin_3); no longer J2.1 (Pin_1)
- net SWDIO: now also J2.1 (Pin_1); no longer J2.3 (Pin_3)
- net USB_CC: now also J1.2 (Pin_2); no longer J1.4 (Pin_4)
- net USB_D-: now also J1.4 (Pin_4); no longer J1.2 (Pin_2)
- net VBUS: now also J1.5 (Pin_5); no longer J1.1 (Pin_1)
- new net: D1.2 (DIN), R3.2
Other:
- moved on the sheet: D1, J1
Changed lines of the file:
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@@
 	)
 	(no_connect
+		(at 186.69 151.13)
+	)
+	(no_connect
 		(at 186.69 100.33)
 	)
@@
 	)
 	(no_connect
-		(at 186.69 77.47)
-	)
-	(no_connect
-		(at 236.22 105.41)
+		(at 248.92 119.38)
 	)
 	(wire
@@
 	(wire
 		(pts
-			(xy 209.55 105.41) (xy 220.98 105.41)
+			(xy 214.63 119.38) (xy 226.06 119.38)
 		)
 		(stroke
@@
 	(wire
 		(pts
+			(xy 231.14 119.38) (xy 233.68 119.38)
+		)
+		(stroke
+			(width 0)
+			(type default)
+		)
+	)
+	(wire
+		(pts
 			(xy 113.03 102.87) (xy 120.65 102.87)
 		)
@@
 	(wire
 		(pts
-			(xy 186.69 151.13) (xy 193.04 151.13)
+			(xy 186.69 77.47) (xy 193.04 77.47)
 		)
 		(stroke
@@
 	)
 	(label "RGB_DIN"
-		(at 193.04 151.13 0)
+		(at 193.04 77.47 0)
 		(effects
 			(font
@@
 	)
 	(label "RGB_DIN"
-		(at 209.55 105.41 0)
+		(at 214.63 119.38 0)
 		(effects
 			(font
@@
 	)
 	(label "SWCLK"
-		(at 33.02 167.64 0)
+		(at 33.02 172.72 0)
 		(effects
 			(font
@@
 	)
 	(label "SWDIO"
-		(at 33.02 172.72 0)
+		(at 33.02 167.64 0)
 		(effects
 			(font
@@
 	(symbol
 		(lib_id "power:+3V3")
-		(at 228.6 97.79 0)
+		(at 241.3 111.76 0)
 		(unit 1)
 		(body_style 1)
@@
 		(fields_autoplaced yes)
 		(property "Reference" "#PWR020"
-			(at 228.6 101.6 0)
+			(at 241.3 115.57 0)
 			(hide yes)
 			(show_name no)
@@
 		)
 		(property "Value" "+3V3"
-			(at 228.6 92.71 0)
+			(at 241.3 106.68 0)
 			(show_name no)
 			(do_not_autoplace no)
@@
 		)
 		(property "Footprint" ""
-			(at 228.6 97.79 0)
+			(at 241.3 111.76 0)
 			(hide yes)
 			(show_name no)
@@
 		)
 		(property "Datasheet" ""
-			(at 228.6 97.79 0)
+			(at 241.3 111.76 0)
 			(hide yes)
 			(show_name no)
@@
 		)
 		(property "Description" "Power symbol creates a global label with name \"+3V3\""
-			(at 228.6 97.79 0)
+			(at 241.3 111.76 0)
 			(hide yes)
 			(show_name no)
@@
 			)
 		)
-		(property "Footprint" "Capacitor_SMD:C_0805_2012Metric"
+		(property "Footprint" "RP2354A:C_0402_1005Metric_small_pads"
 			(at 22.86 81.28 0)
 			(hide yes)
@@
 	(symbol
 		(lib_id "Connector_Generic:Conn_01x05")
-		(at 25.4 36.83 0)
-		(mirror y)
+		(at 25.4 36.83 180)
 		(unit 1)
 		(body_style 1)
@@
 		(dnp no)
 		(property "Reference" "J1"
-			(at 22.86 35.5599 0)
+			(at 22.86 38.1001 0)
 			(show_name no)
 			(do_not_autoplace no)
@@
 		)
 		(property "Value" "USB"
-			(at 22.86 38.0999 0)
+			(at 22.86 35.5601 0)
 			(show_name no)
 			(do_not_autoplace no)
@@
 	(symbol
 		(lib_id "power:GND")
-		(at 228.6 113.03 0)
+		(at 241.3 127 0)
 		(unit 1)
 		(body_style 1)
@@
 		(fields_autoplaced yes)
 		(property "Reference" "#PWR021"
-			(at 228.6 119.38 0)
+			(at 241.3 133.35 0)
 			(hide yes)
 			(show_name no)
@@
 		)
 		(property "Value" "GND"
-			(at 228.6 118.11 0)
+			(at 241.3 132.08 0)
 			(show_name no)
 			(do_not_autoplace no)
@@
 		)
 		(property "Footprint" ""
-			(at 228.6 113.03 0)
+			(at 241.3 127 0)
 			(hide yes)
 			(show_name no)
@@
 		)
 		(property "Datasheet" ""
-			(at 228.6 113.03 0)
+			(at 241.3 127 0)
 			(hide yes)
 			(show_name no)
@@
 		)
 		(property "Description" "Power symbol creates a global label with name \"GND\" , ground"
-			(at 228.6 113.03 0)
+			(at 241.3 127 0)
 			(hide yes)
 			(show_name no)
@@
 	(symbol
 		(lib_id "Device:R_Small")
+		(at 228.6 119.38 90)
+		(unit 1)
+		(body_style 1)
+		(exclude_from_sim no)
+		(in_bom yes)
+		(on_board yes)
+		(in_pos_files yes)
+		(dnp no)
+		(fields_autoplaced yes)
+		(property "Reference" "R3"
+			(at 228.6 114.3 90)
+			(show_name no)
+			(do_not_autoplace no)
+			(effects
+				(font
+					(size 1.016 1.016)
+				)
+			)
+		)
+		(property "Value" "500"
+			(at 228.6 116.84 90)
+			(show_name no)
+			(do_not_autoplace no)
+			(effects
+				(font
+					(size 1.27 1.27)
+				)
+			)
+		)
+		(property "Footprint" "Resistor_SMD:R_0805_2012Metric"
+			(at 228.6 119.38 0)
+			(hide yes)
+			(show_name no)
+			(do_not_autoplace no)
+			(effects
+				(font
+					(size 1.27 1.27)
+				)
+			)
+		)
+		(property "Datasheet" ""
+			(at 228.6 119.38 0)
+			(hide yes)
+			(show_name no)
+			(do_not_autoplace no)
+			(effects
+				(font
+					(size 1.27 1.27)
+				)
+			)
+		)
+		(property "Description" "Resistor, small symbol"
+			(at 228.6 119.38 0)
+			(hide yes)
+			(show_name no)
+			(do_not_autoplace no)
+			(effects
+				(font
+					(size 1.27 1.27)
+				)
+			)
+		)
+		(pin "1"
+		)
+		(pin "2"
+		)
+		(instances
+			(project "beacon"
+				(path "/7a6a2811-0e11-481c-9755-3c5cda6fabc7"
+					(reference "R3")
+					(unit 1)
+				)
+			)
+		)
+	)
+	(symbol
+		(lib_id "Device:R_Small")
 		(at 34.29 41.91 180)
 		(unit 1)
@@
 			)
 		)
-		(property "Footprint" "Resistor_SMD:R_0805_2012Metric"
+		(property "Footprint" "Resistor_SMD:R_0402_1005Metric"
 			(at 34.29 41.91 0)
 			(hide yes)
@@
 			)
 		)
-		(property "Footprint" "Resistor_SMD:R_0805_2012Metric"
+		(property "Footprint" "Resistor_SMD:R_0402_1005Metric"
 			(at 123.19 102.87 0)
 			(hide yes)
@@
 			)
 		)
-		(property "Footprint" "Capacitor_SMD:C_0805_2012Metric"
+		(property "Footprint" "Capacitor_SMD:C_0402_1005Metric"
 			(at 85.09 77.47 0)
 			(hide yes)
@@
 			)
 		)
-		(property "Footprint" "Resistor_SMD:R_0805_2012Metric"
+		(property "Footprint" "Resistor_SMD:R_0402_1005Metric"
 			(at 123.19 100.33 0)
 			(hide yes)
@@
 			)
 		)
-		(property "Footprint" "Capacitor_SMD:C_0805_2012Metric"
+		(property "Footprint" "RP2354A:C_0402_1005Metric_small_pads"
 			(at 33.02 81.28 0)
 			(hide yes)
@@
 	(symbol
 		(lib_id "LED:SK6812")
-		(at 228.6 105.41 0)
+		(at 241.3 119.38 0)
 		(unit 1)
 		(body_style 1)
@@
 		(fields_autoplaced yes)
 		(property "Reference" "D1"
-			(at 238.76 98.9898 0)
+			(at 251.46 112.9598 0)
 			(show_name no)
 			(do_not_autoplace no)
@@
 		)
 		(property "Value" "SK6812"
-			(at 238.76 101.5298 0)
+			(at 251.46 115.4998 0)
 			(show_name no)
 			(do_not_autoplace no)
@@
 		)
 		(property "Footprint" "LED_SMD:LED_SK6812_PLCC4_5.0x5.0mm_P3.2mm"
-			(at 229.87 113.03 0)
+			(at 242.57 127 0)
 			(hide yes)
 			(show_name no)
@@
 		)
 		(property "Datasheet" "https://cdn-shop.adafruit.com/product-files/1138/SK6812+LED+datasheet+.pdf"
-			(at 231.14 114.935 0)
+			(at 243.84 128.905 0)
 			(hide yes)
 			(show_name no)
@@
 		)
 		(property "Description" "RGB LED with integrated controller"
-			(at 228.6 105.41 0)
+			(at 241.3 119.38 0)
 			(hide yes)
 			(show_name no)
@@
 			)
 		)
-		(property "Footprint" "Resistor_SMD:R_0805_2012Metric"
+		(property "Footprint" "Resistor_SMD:R_0402_1005Metric"
 			(at 43.18 68.58 0)
 			(hide yes)
@@
 			)
 		)
-		(property "Footprint" "RP2354A:RP2354A-QFN-60-1EP_7x7mm_P0.4mm_EP3.4x3.4mm"
+		(property "Footprint" "RP2354A:RP2354A-QFN-60-1EP_7x7_P0.4mm_EP3.4x3.4mm_ThermalVias"
 			(at 161.29 115.57 0)
 			(hide yes)
